Commit message: merging in ubi-agni fork

File: flir_ptu_description/urdf/d46.urdf.xacro (robot description, xacro)
@@ -20,20 +20,8 @@
           <color rgba="0.3 0.3 0.3 1.0" />
         </material>
+        <origin xyz="-0.0295 0.011 0" rpy="3.14 0 0" />
         <geometry>
-          <box size="0.045 0.065 0.044" />
+          <mesh filename="package://flir_ptu_description/meshes/flir-ptu-simple.stl"/>
         </geometry>
-        <origin xyz="0 0.011 0" />
-      </visual>
-      <visual>
-        <geometry>
-          <box size="0.046 0.044 0.044" />
-        </geometry>
-        <origin xyz="-0.045 0.0215 0" />
-      </visual>
-      <visual>
-        <geometry>
-          <cylinder length="0.015" radius="0.005" />
-        </geometry>
-        <origin xyz="-0.074 0.021 0" rpy="0 1.57 0" />
       </visual>
       <collision>
@@ -49,11 +37,31 @@
         <origin xyz="-0.045 0.0215 0" />
       </collision>
+      <collision>
+        <geometry>
+          <cylinder length="0.015" radius="0.005" />
+        </geometry>
+        <origin xyz="-0.074 0.021 0" rpy="0 1.57 0" />
+      </collision>
     </link>
+    <gazebo reference="${ptu_name}_${joint_name}_link">
+        <material>Gazebo/DarkGrey</material>
+    </gazebo>
+  </xacro:macro>
+  <xacro:macro name="d46_transmission" params="name">
+    <transmission name="${name}_trans">
+      <type>transmission_interface/SimpleTransmission</type>
+      <joint name="${name}">
+        <hardwareInterface>PositionJointInterface</hardwareInterface>
+      </joint>
+      <actuator name="${name}_motor">
+        <mechanicalReduction>1</mechanicalReduction>
+      </actuator>
+    </transmission>
   </xacro:macro>
   <xacro:macro name="ptu_d46" params="name">
+    <d46_stepper_module ptu_name="${name}" joint_name="pan" />
+    <d46_stepper_module ptu_name="${name}" joint_name="tilt" />
     <link name="${name}_base_link" />
-    <d46_stepper_module ptu_name="${name}" joint_name="pan" />
     <link name="${name}_tilted_link" />
-    <d46_stepper_module ptu_name="${name}" joint_name="tilt" />
     <link name="${name}_mount_link" >
       <inertial>
@@ -115,4 +123,5 @@
       <dynamics friction="10.0" damping="${dynamic_damping}"/>
     </joint>
+    <d46_transmission name="${name}_pan" />
     <!-- The tilt joint -->
     <joint name="${name}_tilt" type="revolute">
@@ -125,4 +134,5 @@
       <dynamics friction="10.0" damping="${dynamic_damping}"/>
     </joint>
+    <d46_transmission name="${name}_tilt" />
     <!-- Fixed joint to provide a convenient attachment point for accessories. -->
     <joint name="${name}_mount" type="fixed">

Commit message: removed unseen visuals

File: flir_ptu_description/urdf/d46.urdf.xacro (robot description, xacro)
@@ -65,46 +65,5 @@
     <link name="${name}_base_link" />
     <link name="${name}_tilted_link" />
-    <link name="${name}_mount_link" >
-      <inertial>
-        <mass value="0.10" />
-        <inertia  ixx="0.00003" ixy="0.0"  ixz="0.0"  iyy="0.00001"  iyz="0.0"	izz="0.00004" />
-      </inertial>
-      <visual>
-        <geometry>
-          <box size="0.025 0.064 0.005" />
-        </geometry>
-        <origin xyz="0.0 0.0 -0.0025" />
-      </visual>
-      <visual>
-        <geometry>
-          <box size="0.025 0.009 0.045" />
-        </geometry>
-       <origin xyz="0.0 0.0275 -0.0275" />
-      </visual>
-      <visual>
-        <geometry>
-          <box size="0.025 0.009 0.045" />
-        </geometry>
-         <origin xyz="0.0 -0.0275 -0.0275" />
-      </visual>
-      <collision>
-        <geometry>
-          <box size="0.025 0.064 0.005" />
-        </geometry>
-        <origin xyz="0.0 0.0 -0.0025" />
-      </collision>
-      <collision>
-        <geometry>
-          <box size="0.025 0.009 0.045" />
-        </geometry>
-        <origin xyz="0.0 0.0275 -0.0275" />
-      </collision>
-      <collision>
-        <geometry>
-          <box size="0.025 0.009 0.045" />
-        </geometry>
-        <origin xyz="0.0 -0.0275 -0.0275" />
-      </collision>
-    </link>
+    <link name="${name}_mount_link" />
     <!-- There's an offset between the origin of the pan joint and the origin of
          the overall device, which is between the mounting screws on its base. -->
